Commit message: modify robot

File: my_robot/urdf/my_robot.xacro (robot description, xacro)
@@ -13,4 +13,9 @@
   <gazebo reference="camera">
     <material>Gazebo/Blue</material>
+  </gazebo>
+  <gazebo reference="front_caster">
+    <mu1>0.0</mu1>
+    <mu2>0.0</mu2>
+    <material>Gazebo/RedBright</material>
   </gazebo>
   <link name="robot_footprint"></link>
@@ -43,6 +48,16 @@
       </geometry>
     </visual>
+  </link>
+  <link name="front_caster">
+    <inertial>
+      <mass value="0.1"/>
+      <origin xyz="0 0 0" rpy="0 0 0"/>
+      <inertia
+	  ixx="1e-6" ixy="0" ixz="0"
+	  iyy="1e-6" iyz="0"
+	  izz="1e-6"/>
+    </inertial>
     <collision name='front_caster_collision'>
-      <origin xyz="0.15 0 -0.1" rpy=" 0 0 0"/>
+      <origin xyz="0 0 0" rpy=" 0 0 0"/>
       <geometry>
         <sphere radius="0.0999"/>
@@ -50,5 +65,5 @@
     </collision>
     <visual name='front_caster_visual'>
-      <origin xyz="0.15 0 -0.1" rpy=" 0 0 0"/>
+      <origin xyz="0 0 0" rpy=" 0 0 0"/>
       <geometry>
         <sphere radius="0.1"/>
@@ -56,4 +71,10 @@
     </visual>
   </link>
+  <joint type="fixed" name="front_caster_joint">
+    <origin xyz="0.15 0 -0.1" rpy="0 0 0"/>
+    <parent link="chassis"/>
+    <child link="front_caster"/>
+    <axis xyz="0 1 0" rpy="0 0 0"/>
+  </joint>
   <link name='left_wheel'>
     <inertial>

Commit message: add rear caster

File: my_robot/urdf/my_robot.xacro (robot description, xacro)
@@ -19,4 +19,9 @@
     <material>Gazebo/RedBright</material>
   </gazebo>
+  <gazebo reference="rear_caster">
+    <mu1>0.0</mu1>
+    <mu2>0.0</mu2>
+    <material>Gazebo/RedBright</material>
+  </gazebo>
   <link name="robot_footprint"></link>
   <joint name="robot_footprint_joint" type="fixed">
@@ -77,4 +82,32 @@
     <axis xyz="0 1 0" rpy="0 0 0"/>
   </joint>
+  <link name="rear_caster">
+    <inertial>
+      <mass value="0.1"/>
+      <origin xyz="0 0 0" rpy="0 0 0"/>
+      <inertia
+	  ixx="1e-6" ixy="0" ixz="0"
+	  iyy="1e-6" iyz="0"
+	  izz="1e-6"/>
+    </inertial>
+    <collision name='rear_caster_collision'>
+      <origin xyz="0 0 0" rpy=" 0 0 0"/>
+      <geometry>
+        <sphere radius="0.0999"/>
+      </geometry>
+    </collision>
+    <visual name='rear_caster_visual'>
+      <origin xyz="0 0 0" rpy=" 0 0 0"/>
+      <geometry>
+        <sphere radius="0.1"/>
+      </geometry>
+    </visual>
+  </link>
+  <joint type="fixed" name="rear_caster_joint">
+    <origin xyz="-0.15 0 -0.1" rpy="0 0 0"/>
+    <parent link="chassis"/>
+    <child link="rear_caster"/>
+    <axis xyz="0 1 0" rpy="0 0 0"/>
+  </joint>
   <link name='left_wheel'>
     <inertial>
@@ -100,5 +133,5 @@
   </link>
   <joint type="continuous" name="left_wheel_hinge">
-    <origin xyz="-0.15 0.22 0" rpy="0 0 0"/>
+    <origin xyz="0 0.22 0" rpy="0 0 0"/>
     <child link="left_wheel"/>
     <parent link="chassis"/>
@@ -130,5 +163,5 @@
   </link>
   <joint type="continuous" name="right_wheel_hinge">
-    <origin xyz="-0.15 -0.22 0" rpy="0 0 0"/>
+    <origin xyz="0 -0.22 0" rpy="0 0 0"/>
     <child link="right_wheel"/>
     <parent link="chassis"/>
